File: LogicBoard 3GE/LogicBoard 3GE.kicad_pcb (KiCad board)
At the start: 4 copper layers, 103.1 x 140.1 mm, 169 parts, among them IC103 LM386-3, IC201 2363, IC202 74LS00, IC203 74LS32, IC204 2114, IC205 2114, IC206 68A09, IC207 6522, IC208 AY3-8912, IC301 MC1408, IC302 CD4052B, IC303 LF347, IC304 LF353, IC305 4066, J103 Conn_01x02, J201 CART, J202 MD-90SM, J203 MD-90SM, J204 Power, J301 Video, J304 Conn_01x03_Pin, Q301 FMMT3905, Q302 FMMT3905, Q303 FMMT3904, SW201 RESET BUTTON, Y201 6MHz

Commit message: Remove all tracks, change RAM, change ROM, change electrolitic caps
Parts:
- removed C201, C205: 0.1uF, Capacitor_SMD:C_0805_2012Metric
- removed IC205: 2114, Package_DIP:DIP-18_W7.62mm
- added C1: 0.1uF, Capacitor_SMD:C_0805_2012Metric, F.Cu at (137.3, 94.9)
- C113: footprint Capacitor_SMD:CP_Elec_4x5.3 -> Capacitor_Tantalum_SMD:CP_EIA-7260-15_AVX-R_Pad2.68x6.30mm_HandSolder
- C114: footprint Capacitor_SMD:CP_Elec_8x10.5 -> Capacitor_Tantalum_SMD:CP_EIA-7260-15_AVX-R_Pad2.68x6.30mm_HandSolder
- C211, C212, C213: footprint Capacitor_SMD:CP_Elec_8x6.5 -> Capacitor_Tantalum_SMD:CP_EIA-3528-15_AVX-H
- IC201: value 2363 -> 27C512PLCC; footprint Package_DIP:DIP-28_W15.24mm -> Package_LCC:PLCC-32_11.4x14.0mm_P1.27mm
- IC204: value 2114 -> CY62256-70PC; footprint Package_DIP:DIP-18_W7.62mm -> Package_SO:SOP-28_8.4x18.16mm_P1.27mm
- J201: value CART -> AMP 5645384-1
- SW201: value RESET BUTTON -> Conn_01x02
- moved D301 183.0 mm to (-83.5, 64.6)
- moved R207 183.0 mm to (-73.7, 65.7)
- moved R314 183.0 mm to (-78.8, 64.6)
- moved D201 133.6 mm to (-0.27, 47.1)
- moved R206 133.6 mm to (-19.0, 47.5)
- moved R214 133.6 mm to (-15.2, 47.3)
- moved R215 133.6 mm to (-11.3, 47.3)
- moved R226 133.6 mm to (-22.8, 47.5)
- moved R341 133.6 mm to (7.41, 41.5)
- moved R342 133.6 mm to (-4.16, 47.2)
- moved R343 133.6 mm to (-7.65, 47.3)
- moved R344 133.6 mm to (-3.40, 41.5)
- moved R345 133.6 mm to (0.38, 41.5)
- moved R346 133.6 mm to (3.94, 41.4)
- moved C227 132.2 mm to (-56.3, 42.9)
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Connections:
- C106 pad 1: Net-(IC103-+) -> /~{RESET}
- C114 pad 2: Net-(J103-Pin_1) -> /~{RESET}
- C116 pad 1: Net-(C116-Pad1) -> /~{RESET}
- IC103 pad 1: unconnected-(IC103-GAIN-Pad1) -> /~{RESET}
- IC103 pad 2: GND -> /~{RESET}
- IC103 pad 3: Net-(IC103-+) -> /~{RESET}
- IC103 pad 4: GND -> /~{RESET}
- IC201 pad 1: +5V -> unconnected-(IC201-NC-Pad1)
- IC201 pad 10: /A0 -> /A1
- IC201 pad 11: /D0 -> /A0
- IC201 pad 12: /D1 -> unconnected-(IC201-NC-Pad12)
- IC201 pad 13: /D2 -> /D0
- IC201 pad 14: GND -> /D1
- IC201 pad 15: /D3 -> /D2
- IC201 pad 16: /D4 -> GND
- IC201 pad 17: /D5 -> unconnected-(IC201-NC-Pad17)
- IC201 pad 18: /D6 -> /D3
- IC201 pad 19: /D7 -> /D4
- IC201 pad 2: /A12 -> GND
- IC201 pad 20: /~{ROMS} -> /D5
- IC201 pad 21: /A10 -> /D6
- IC201 pad 22: /~{ROMOE} -> /D7
- IC201 pad 23: /A11 -> /~{ROMOE}
- IC201 pad 24: /A9 -> /A10
- IC201 pad 25: /A8 -> /~{ROMS}
- IC201 pad 27: +5V -> /A11
- IC201 pad 28: +5V -> /A9
- IC201 pad 3: /A7 -> /A12
- IC201 pad 4: /A6 -> /A7
- IC201 pad 5: /A5 -> /A6
- IC201 pad 6: /A4 -> /A5
- IC201 pad 7: /A3 -> /A4
- IC201 pad 8: /A2 -> /A3
- IC201 pad 9: /A1 -> /A2
- IC204 pad 1: /A6 -> GND
- IC204 pad 10: /RAM_R~{W} -> /A0
- IC204 pad 11: /D3 -> /D0
- IC204 pad 12: /D2 -> /D1
- IC204 pad 13: /D1 -> /D2
- IC204 pad 14: /D0 -> GND
- IC204 pad 15: /A9 -> /D3
- IC204 pad 16: /A8 -> /D4
- IC204 pad 17: /A7 -> /D5
- IC204 pad 18: +5V -> /D6
- IC204 pad 2: /A5 -> GND
- IC204 pad 3: /A4 -> /A7
- IC204 pad 4: /A3 -> /A6
- IC204 pad 5: /A0 -> /A5
- IC204 pad 6: /A1 -> /A4
- IC204 pad 7: /A2 -> /A3
- IC204 pad 8: /~{RAMS} -> /A2
- IC204 pad 9: GND -> /A1
- J103 pad 1: Net-(J103-Pin_1) -> /~{RESET}
- R103 pad 1: Net-(C116-Pad1) -> /~{RESET}
- R104 pad 2: Net-(IC103-+) -> /~{RESET}
- R105 pad 2: Net-(IC103-+) -> /~{RESET}
Routing:
- net GND: track 943.4 -> 0.00 mm, vias 34 -> 0
- net +5V: track 621.5 -> 10.2 mm, vias 64 -> 5
- net /~{ROMS}: track 237.6 -> 0.00 mm, vias 7 -> 0
- net /A6: track 201.6 -> 3.00 mm, vias 2 -> 0
- net /A9: track 191.8 -> 0.00 mm, vias 2 -> 0
- net /A0: track 184.2 -> 0.00 mm, vias 2 -> 0
- net /A8: track 182.8 -> 0.00 mm, vias 4 -> 0
- net /A7: track 176.3 -> 3.00 mm, vias 2 -> 0
- net /A3: track 175.6 -> 3.03 mm, vias 1 -> 0
- net -5VA: track 170.3 -> 0.00 mm, vias 8 -> 0
- net Net-(C114-Pad1): track 183.2 -> 16.0 mm, vias 3 -> 0
- net /A5: track 163.1 -> 3.03 mm
- net /SW7: track 155.1 -> 0.00 mm, vias 3 -> 0
- net /A1: track 156.0 -> 3.03 mm, vias 1 -> 0
- net /CH(A+B+C): track 150.2 -> 0.00 mm, vias 2 -> 0
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- added copper zone on In1.Cu, net GND
- removed copper zone on B.Cu, net +5V
- removed copper zone on F.Cu, net +5V
- removed copper zone on In1.Cu, net +5V

Commit message: iteration 2
Parts:
- added REF**: FailMaker, VectrexLibrary:FailMaker, F.Cu at (91.7, 136.0)
- C304↓: renamed from C304; moved to F.Cu
- C305↓: renamed from C305; moved to F.Cu
- C306↓: renamed from C306; moved to F.Cu
- C312↓: renamed from C312; moved to F.Cu
- C313↓: renamed from C313; moved to F.Cu
- moved R203 205.6 mm to (148.3, 100.2)
- moved R202 202.2 mm to (148.3, 94.4), turned to 90 degrees
- moved C320 200.4 mm to (120.2, 141.2), turned to -90 degrees
- moved D301 195.0 mm to (111.4, 69.3), turned to 90 degrees
- moved C202 194.6 mm to (117.5, 145.1)
- moved IC302 194.1 mm to (143.9, 141.1), turned to -90 degrees
- moved R314 193.6 mm to (114.7, 69.4), turned to 90 degrees
- moved C325 193.1 mm to (138.7, 152.1), turned to 90 degrees
- moved C314 192.1 mm to (117.6, 141.2), turned to -90 degrees
- moved IC303 190.8 mm to (144.3, 130.0)
- moved Q302 186.3 mm to (129.2, 141.2), turned to 0 degrees
- moved C204 182.7 mm to (114.4, 136.5)
- moved C209 181.3 mm to (127.0, 136.4)
- moved C236 180.7 mm to (124.5, 136.4)
- moved R206 180.6 mm to (147.0, 118.7)
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- renumbered C113 to C113↓, C114 to C114↑, C203 to C203↓, C228 to C228↑, C302 to C302↓, IC305 to IC305↓, Q301 to Q301↓, R320 to R320→, R201 to ←R201, R305 to ↑R305, R338 to ↑R338, R340 to ↑R340, R316 to →R316, R317 to →R317, R318 to →R318, R319 to →R319, R322 to →R322, R323 to →R323, C303 to ↓C303
Connections:
- C106 pad 1: /~{RESET} -> Net-(IC103-+)
- C114↑ pad 2: /~{RESET} -> Net-(J103-Pin_1)
- C116 pad 1: /~{RESET} -> Net-(C116-Pad1)
- IC103 pad 1: /~{RESET} -> unconnected-(IC103-GAIN-Pad1)
- IC103 pad 2: /~{RESET} -> GND
- IC103 pad 3: /~{RESET} -> Net-(IC103-+)
- IC103 pad 4: /~{RESET} -> GND
- J103 pad 1: /~{RESET} -> Net-(J103-Pin_1)
- R103 pad 1: /~{RESET} -> Net-(C116-Pad1)
- R104 pad 2: /~{RESET} -> Net-(IC103-+)
- R105 pad 2: /~{RESET} -> Net-(IC103-+)
Routing:
- net +5V: track 10.2 -> 640.7 mm, vias 5 -> 11
- net -5VA: track 0.00 -> 364.0 mm, vias 0 -> 5
- net GND: track 0.00 -> 284.7 mm, vias 0 -> 38
- net /IC303D_FB: track 0.00 -> 217.8 mm, vias 0 -> 3
- net /A0: track 0.00 -> 212.0 mm, vias 0 -> 3
- net /X2: track 0.00 -> 200.4 mm, vias 0 -> 3
- net /SW7: track 0.00 -> 195.6 mm, vias 0 -> 2
- net /A1: track 3.03 -> 190.3 mm, vias 0 -> 1
- net /IC303A_FB: track 0.00 -> 185.2 mm, vias 0 -> 3
- net /X1: track 0.00 -> 183.3 mm, vias 0 -> 2
- net /VOUT: track 0.00 -> 178.5 mm, vias 0 -> 4
- net /SW1: track 0.00 -> 171.4 mm, vias 0 -> 1
- net /SW2: track 0.00 -> 159.0 mm, vias 0 -> 1
- net /A3: track 3.03 -> 159.5 mm, vias 0 -> 2
- net /A4: track 3.00 -> 154.1 mm, vias 0 -> 3
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- added copper zone on In2.Cu, net GND
- removed copper zone on In2.Cu, net +5V
- removed copper zone on In1.Cu, net -5VA
Other:
- board text added: "VECTREX MICRO V1.1"
- board text removed: "VECTREX MICRO V1.0"
