File: DeflectionBoard/DeflectionBoard.kicad_pcb (KiCad board)
At the start: 2 copper layers, 100 x 100 mm, 97 parts, among them J1 Conn_01x04, J101 Conn_01x02, J201 YOKE, J301 YOKE, U101 TPS55340PWPR, U102 AP63205WU, U103 REF3325AIDCKT, U201 CSD97394Q4M, U202 CSD97394Q4M, U203 INA240A1D, U204 OPA2196xD, U205 TLV3501AID, U206 74LVC1G04, U207 74LVC1G08, U208 74LVC1G08, U301 CSD97394Q4M, U302 CSD97394Q4M, U303 INA240A1D, U304 OPA2196xD, U305 TLV3501AID, U306 74LVC1G04, U307 74LVC1G08, U308 74LVC1G08

Commit message: Checkpoint before project rename to MicroDeflect
Parts:
- moved J1 12.7 mm to (104.3, 51.5)
Routing:
- net /Deflection_Channel_Y/AXIS_IN: track 138.8 -> 150.3 mm
- net /Deflection_Channel_X/AXIS_IN: track 114.4 -> 125.4 mm
- net GND: track 197.5 -> 187.0 mm, vias 76 -> 75
Other:
- board text added: "Channel X"
- board text added: "Channel Y"
- board text added: "Power Boost"
- board text added: "Vectrex Micro MicroDeflect Board v1.0 2026 Daniel Ferrer"
Changed lines of the file:
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@@
 	(footprint "Connector_JST:JST_PH_B4B-PH-K_1x04_P2.00mm_Vertical"
 		(layer "F.Cu")
-		(at 116.9596 53.1786)
+		(at 104.34 51.47)
 		(descr "JST PH series connector, B4B-PH-K (http://www.jst-mfg.com/product/pdf/eng/ePH.pdf)")
 		(tags "connector JST PH vertical")
@@
 	)
 	(gr_rect
+		(start 99.685 106.42)
+		(end 195.235 128.73)
+		(stroke
+			(width 0.2)
+			(type solid)
+		)
+		(fill no)
+		(layer "F.SilkS")
+	)
+	(gr_rect
+		(start 99.94 82.17)
+		(end 195.49 104.34)
+		(stroke
+			(width 0.2)
+			(type solid)
+		)
+		(fill no)
+		(layer "F.SilkS")
+	)
+	(gr_rect
+		(start 99.98 46.56)
+		(end 195.53 80.58)
+		(stroke
+			(width 0.2)
+			(type solid)
+		)
+		(fill no)
+		(layer "F.SilkS")
+	)
+	(gr_rect
 		(start 97.5868 37.4904)
 		(end 197.5868 137.4904)
@@
 		(layer "Edge.Cuts")
 	)
+	(gr_text "Power Boost"
+		(at 142.228571 49.71 0)
+		(layer "F.SilkS")
+		(effects
+			(font
+				(size 1.5 1.5)
+				(thickness 0.3)
+				(bold yes)
+			)
+			(justify left bottom)
+		)
+	)
+	(gr_text "Channel Y"
+		(at 143.45 108.99 0)
+		(layer "F.SilkS")
+		(effects
+			(font
+				(size 1.5 1.5)
+				(thickness 0.3)
+				(bold yes)
+			)
+			(justify left bottom)
+		)
+	)
+	(gr_text "Channel X"
+		(at 143.7 84.98 0)
+		(layer "F.SilkS")
+		(effects
+			(font
+				(size 1.5 1.5)
+				(thickness 0.3)
+				(bold yes)
+			)
+			(justify left bottom)
+		)
+	)
+	(gr_text "Vectrex Micro\n\nMicroDeflect Board v1.0\n\n2026 Daniel Ferrer"
+		(at 165.43 60.44 0)
+		(layer "F.SilkS")
+		(effects
+			(font
+				(size 1.5 1.5)
+				(thickness 0.3)
+				(bold yes)
+			)
+			(justify left bottom)
+		)
+	)
 	(segment
 		(start 155.4754 90.957398)
@@
 	)
 	(via
-		(at 146.93 105.37)
+		(at 146.9567 105.37)
 		(size 0.6)
 		(drill 0.3)
@@
 	)
 	(segment
-		(start 136.24 111.08)
-		(end 141.95 105.37)
-		(width 0.8)
-		(layer "B.Cu")
-		(net "+5V")
-	)
-	(segment
 		(start 164.0104 99.492398)
 		(end 166.7504 99.492398)
@@
 	)
 	(segment
-		(start 146.93 105.37)
-		(end 146.9567 105.37)
-		(width 0.8)
-		(layer "B.Cu")
-		(net "+5V")
-	)
-	(segment
 		(start 121.0375 112.757398)
 		(end 131.4675 112.757398)
@@
 	(segment
 		(start 141.95 105.37)
-		(end 146.93 105.37)
+		(end 136.24 111.08)
 		(width 0.8)
 		(layer "B.Cu")
@@
 	)
 	(segment
+		(start 146.9567 105.37)
+		(end 141.95 105.37)
+		(width 0.8)
+		(layer "B.Cu")
+		(net "+5V")
+	)
+	(segment
 		(start 145.1504 70.322398)
 		(end 143.7204 71.752398)
@@
 	)
 	(segment
-		(start 125.662202 59.892398)
-		(end 126.0896 59.465)
-		(width 0.5)
-		(layer "F.Cu")
-		(net "GND")
-	)
-	(segment
 		(start 128.8589 73.685034)
 		(end 129.880666 73.685034)
@@
 	)
 	(segment
-		(start 124.7804 59.892398)
-		(end 125.662202 59.892398)
-		(width 0.5)
-		(layer "F.Cu")
-		(net "GND")
-	)
-	(segment
 		(start 158.71 121.4)
 		(end 159.13 121.82)
@@
 	)
 	(via
-		(at 124.7804 59.892398)
-		(size 0.6)
-		(drill 0.3)
-		(layers "F.Cu" "B.Cu")
-		(net "GND")
-	)
-	(via
 		(at 146.2075 121.107398)
 		(size 0.6)
@@
 	)
 	(via
-		(at 126.0896 59.465)
+		(at 124.7804 59.892398)
 		(size 0.6)
 		(drill 0.3)
@@
 	)
 	(segment
-		(start 123.1054 60.427398)
-		(end 124.2454 60.427398)
-		(width 0.5)
-		(layer "B.Cu")
-		(net "GND")
-	)
-	(segment
 		(start 117.38 113.09)
 		(end 119.17 114.88)
@@
 	)
 	(segment
-		(start 124.2454 60.427398)
-		(end 124.7804 59.892398)
-		(width 0.5)
-		(layer "B.Cu")
-		(net "GND")
-	)
-	(segment
 		(start 157.2804 99.832398)
 		(end 158.1104 99.832398)
@@
 	)
 	(segment
-		(start 122.9596 60.281598)
-		(end 122.9596 53.1786)
-		(width 0.5)
-		(layer "B.Cu")
-		(net "GND")
-	)
-	(segment
 		(start 143.48 75.46)
 		(end 143.5 75.44)
@@
 	)
 	(segment
-		(start 121.567602 46.132398)
-		(end 158.7504 46.132398)
-		(width 1)
-		(layer "F.Cu")
-		(net "/Deflection_Channel_X/AXIS_IN")
-	)
-	(segment
-		(start 194.7704 93.900296)
-		(end 190.8104 97.860296)
+		(start 190.8104 97.860296)
+		(end 194.7704 93.900296)
 		(width 1)
 		(layer "F.Cu")
@@
 	)
 	(segment
-		(start 116.9596 53.1786)
-		(end 116.9596 50.7404)
+		(start 108.802602 46.132398)
+		(end 104.34 50.595)
 		(width 1)
 		(layer "F.Cu")
@@
 	(segment
 		(start 158.7504 46.132398)
-		(end 182.6804 70.062398)
+		(end 108.802602 46.132398)
 		(width 1)
 		(layer "F.Cu")
@@
 	)
 	(segment
-		(start 182.6804 70.062398)
+		(start 194.7704 93.900296)
 		(end 194.7704 82.152398)
 		(width 1)
@@
 	)
 	(segment
-		(start 194.7704 82.152398)
-		(end 194.7704 93.900296)
+		(start 104.34 50.595)
+		(end 104.34 51.47)
 		(width 1)
 		(layer "F.Cu")
@@
 	)
 	(segment
-		(start 116.9596 50.7404)
-		(end 121.567602 46.132398)
+		(start 194.7704 82.152398)
+		(end 158.7504 46.132398)
 		(width 1)
 		(layer "F.Cu")
@@
 	)
 	(segment
-		(start 120.22 50.9)
-		(end 118.9596 52.1604)
-		(width 1)
-		(layer "B.Cu")
-		(net "/Deflection_Channel_Y/AXIS_IN")
-	)
-	(segment
-		(start 162.65 47.2)
-		(end 123.92 47.2)
+		(start 110.335 47.2)
+		(end 106.34 51.195)
 		(width 1.2)
 		(layer "B.Cu")
@@
 	)
 	(segment
-		(start 123.92 47.2)
-		(end 120.22 50.9)
-		(width 1)
+		(start 106.34 51.195)
+		(end 106.34 51.47)
+		(width 1.2)
 		(layer "B.Cu")
 		(net "/Deflection_Channel_Y/AXIS_IN")
 	)
 	(segment
-		(start 118.9596 52.1604)
-		(end 118.9596 53.1786)
-		(width 1)
+		(start 162.65 47.2)
+		(end 110.335 47.2)
+		(width 1.2)
 		(layer "B.Cu")
 		(net "/Deflection_Channel_Y/AXIS_IN")
