File: MicroDeflect/MicroDeflect.kicad_pcb (KiCad board)
At the start: 2 copper layers, 100 x 100 mm, 97 parts, among them J1 Conn_01x04, J101 Conn_01x02, J201 YOKE, J301 YOKE, U101 TPS55340PWPR, U102 AP63205WU, U103 REF3325AIDCKT, U201 CSD97394Q4M, U202 CSD97394Q4M, U203 INA240A1D, U204 OPA2196xD, U205 TLV3501AID, U206 74LVC1G04, U207 74LVC1G08, U208 74LVC1G08, U301 CSD97394Q4M, U302 CSD97394Q4M, U303 INA240A1D, U304 OPA2196xD, U305 TLV3501AID, U306 74LVC1G04, U307 74LVC1G08, U308 74LVC1G08

Commit message: Clean up KiCad rename artifacts; MicroDeflect is the project
Remove stray DeflectionBoard.* files and _restore_backup that KiCad
recreated when the old project was still open during the rename.
MicroDeflect.* (latest, 21:16) is the real work; project validated.

Co-Authored-By: Claude Opus 4.8 <noreply@anthropic.com>
Parts:
- moved J101 12.1 mm to (105.5, 75.7)
- moved J1 7.82 mm to (108.7, 58.0), turned to -90 degrees
Connections:
- J1 pad 3: Z_AXIS -> EN
Routing:
- net EN: track 58.3 -> 147.3 mm
- net /Deflection_Channel_Y/AXIS_IN: track 150.3 -> 179.1 mm, vias 2 -> 0
- net GND: track 187.0 -> 191.3 mm
- net /Deflection_Channel_X/AXIS_IN: track 125.4 -> 128.2 mm
- net Net-(D101-A): track 13.1 -> 15.5 mm
Other:
- board text added: "GND"
- board text added: "Input"
- board text added: "Power In"
- board text added: "X"
- board text added: "X Center"
- board text added: "X Gain"
- board text added: "X Yoke"
- board text added: "Y"
- board text added: "Y Yoke"
- board text added: "Z"

Commit message: MicroDeflect: add J2 (HV board interface), fix J1.3 = Z_AXIS
- J1.3 restored to Z_AXIS (was wrongly on EN); J1 = LogicBoard input (X/Y/Z/GND)
- J2 added = output to HV board: Z_AXIS (pass-through from J1.3), GND, EN
- EN net (R208 pull-up + AND gates) routed to J2.3 for HV spot-killer disable
- DRC: 0 unconnected (J2 placed + routed)

Co-Authored-By: Claude Opus 4.8 <noreply@anthropic.com>
Parts:
- added J2: Conn_01x03, Connector_JST:JST_PH_B3B-PH-K_1x03_P2.00mm_Vertical, F.Cu at (192.3, 61.8)
- H301, H302, H303, H304: footprint MountingHole:MountingHole_3.2mm_M3_DIN965_Pad -> MountingHole:MountingHole_3mm
Connections:
- J1 pad 3: EN -> Z_AXIS
Routing:
- net Z_AXIS: track 0.00 -> 111.9 mm
- net EN: track 147.3 -> 108.8 mm, vias 9 -> 13
- net /Deflection_Channel_Y/AXIS_IN: track 179.1 -> 178.8 mm, vias 0 -> 1
Other:
- board text added: "EN"
- board text added: "Output"
