File: LogicBoard 3GE Repro/LogicBoard 3GE Repro.kicad_pcb (KiCad board)
At the start: 2 copper layers, 93 parts, among them IC201 2363, IC204 2114, IC205 2114, IC206 68A09, IC207 6522, IC208 AY3-8912, IC301 MC1408, IC302 CD4052B, IC303 LF347, IC304 LF353, IC305 4066, J204 Power, J301 Video, J302 Audio, Q301 2N3905, Q302 2N3905, Q303 2N3904, SW201 Reset, U1 ATF16V8Bxx-xxPU

Commit message: Repro: remove redundant R326 volume pot (volume now single, in preamp)
R326 was the original Vectrex preamp volume pot; redundant now that the
external panel pot (J304) does it. Removed R326, merged the channel-mix
node into AUDIO -> J304 -> LM386. 3 calibration trimmers remain
(R302/R333/R335). ERC 11.

Co-Authored-By: Claude Opus 4.8 <noreply@anthropic.com>
Parts:
- removed C205: 0.1uF, Capacitor_THT:C_Disc_D5.0mm_W2.5mm_P5.00mm
- removed C210, C222: 20pF, Capacitor_THT:C_Disc_D5.0mm_W2.5mm_P5.00mm
- removed C238: 10uF 16V, Capacitor_THT:CP_Radial_Tantal_D5.0mm_P2.50mm
- removed IC205: 2114, Package_DIP:DIP-18_W7.62mm
- removed J302: Audio, Connector_Molex:Molex_KK-254_AE-6410-02A_1x02_P2.54mm_Vertical
- removed U1: ATF16V8Bxx-xxPU, Package_DIP:DIP-20_W7.62mm
- added C1: 0.1uF, Capacitor_SMD:C_0402_1005Metric, F.Cu at (102.8, 76.4)
- added C2: 0.1uF, Capacitor_SMD:C_0402_1005Metric, F.Cu at (120.2, 72.6)
- added C329: 0.1uF, Capacitor_SMD:C_0402_1005Metric, F.Cu at (146.0, 130.4)
- added C330: 10uF, Capacitor_SMD:C_0402_1005Metric, F.Cu at (147.3, 140.0)
- added C331: 0.1uF, Capacitor_SMD:C_0402_1005Metric, F.Cu at (145.3, 140.0)
- added C332: C_Polarized_Small, Capacitor_SMD:CP_Elec_8x10.5, F.Cu at (128.1, 135.0)
- added C333: 47nF, Capacitor_SMD:C_0402_1005Metric, F.Cu at (143.3, 140.1)
- added IC202: ATF16V8Bxx-xxPU, Package_SO:SOIC-20W_7.5x12.8mm_P1.27mm, F.Cu at (87.0, 80.8)
- added IC209: 74HC74, Package_SO:SOIC-14_3.9x8.7mm_P1.27mm, F.Cu at (118.5, 77.3)
- added IC306: LM386, Package_SO:SOIC-8_3.9x4.9mm_P1.27mm, F.Cu at (141.7, 135.3)
- added J201: CART, Vectrex LogicBoard:SULLINS_EBC18DRAS, F.Cu at (137.5, 38.2)
- added J202: DB9_Male, Vectrex LogicBoard:DSUB-9_Male_Horizontal_Vectrex, F.Cu at (92.6, 142.8)
- added J203: DB9_Male, Vectrex LogicBoard:DSUB-9_Male_Horizontal_Vectrex, F.Cu at (127.6, 142.9)
- added J303: Speaker, Connector_PinHeader_2.54mm:PinHeader_1x02_P2.54mm_Vertical, F.Cu at (152.5, 143.0)
- added J304: Volume, Connector_PinHeader_2.54mm:PinHeader_1x03_P2.54mm_Vertical, F.Cu at (151.1, 137.6)
- added JP1: Jumper_3_Bridged12, Connector_PinHeader_2.54mm:PinHeader_1x03_P2.54mm_Vertical, F.Cu at (55.2, 43.7)
- added JP2: Jumper_3_Bridged12, Connector_PinHeader_2.54mm:PinHeader_1x03_P2.54mm_Vertical, F.Cu at (59.8, 43.7)
- added JP3: Jumper_3_Bridged12, Connector_PinHeader_2.54mm:PinHeader_1x03_P2.54mm_Vertical, F.Cu at (64.4, 43.7)
- added R201: 22k, Resistor_SMD:R_0402_1005Metric, F.Cu at (92.6, 97.7)
- added R202: 3.3k, Resistor_SMD:R_0402_1005Metric, F.Cu at (-100.3, 5.63)
- added R203: 3.3k, Resistor_SMD:R_0402_1005Metric, F.Cu at (-100.3, 9.68)
- added R204: 3.3k, Resistor_SMD:R_0402_1005Metric, F.Cu at (-223.1, 198.3)
- added R205: 3.3k, Resistor_SMD:R_0402_1005Metric, F.Cu at (79.1, 151.2)
- added R206: 3.3k, Resistor_SMD:R_0402_1005Metric, F.Cu at (-100.3, 21.8)
- added R207: 3.3k, Resistor_SMD:R_0402_1005Metric, F.Cu at (-100.3, 25.9)
- added R208: 100, Resistor_SMD:R_0402_1005Metric, F.Cu at (92.6, 91.3)
- added R214: 33, Resistor_SMD:R_0402_1005Metric, F.Cu at (-100.3, 42.1)
- added R215: 33, Resistor_SMD:R_0402_1005Metric, F.Cu at (-100.3, 46.1)
- added R216: 33, Resistor_SMD:R_0402_1005Metric, F.Cu at (-100.3, 50.2)
- added R217: 33, Resistor_SMD:R_0402_1005Metric, F.Cu at (-100.3, 54.2)
- added R218: 680, Resistor_SMD:R_0402_1005Metric, F.Cu at (-214.0, 212.6)
- added R219: 680, Resistor_SMD:R_0402_1005Metric, F.Cu at (-214.0, 216.6)
- added R220: 680, Resistor_SMD:R_0402_1005Metric, F.Cu at (-207.2, 186.2)
- added R221: 680, Resistor_SMD:R_0402_1005Metric, F.Cu at (-207.2, 190.2)
- added R222: 680, Resistor_SMD:R_0402_1005Metric, F.Cu at (-207.2, 194.3)
- added R223: 680, Resistor_SMD:R_0402_1005Metric, F.Cu at (-207.2, 198.3)
- added R224: 680, Resistor_SMD:R_0402_1005Metric, F.Cu at (-207.2, 202.4)
- added R225: 680, Resistor_SMD:R_0402_1005Metric, F.Cu at (-207.2, 206.4)
- added R301: 2.7k 1%, Resistor_SMD:R_0402_1005Metric, F.Cu at (-84.5, 25.9)
- added R303: 3.6k 1%, Resistor_SMD:R_0402_1005Metric, F.Cu at (-84.5, 29.9)
- added R304: 2.7k 1%, Resistor_SMD:R_0402_1005Metric, F.Cu at (-84.5, 34.0)
- added R305: 2.7k 1%, Resistor_SMD:R_0402_1005Metric, F.Cu at (-84.5, 38.0)
- added R306: 680, Resistor_SMD:R_0402_1005Metric, F.Cu at (79.1, 148.3)
- added R307: 330k, Resistor_SMD:R_0402_1005Metric, F.Cu at (79.1, 155.5)
- added R308: 680, Resistor_SMD:R_0402_1005Metric, F.Cu at (79.1, 149.8)
- added R309: 330k, Resistor_SMD:R_0402_1005Metric, F.Cu at (79.0, 158.3)
- added R310: 680, Resistor_SMD:R_0402_1005Metric, F.Cu at (-198.1, 212.6)
- added R311: 330k, Resistor_SMD:R_0402_1005Metric, F.Cu at (-198.1, 216.6)
- added R312: 680, Resistor_SMD:R_0402_1005Metric, F.Cu at (-191.4, 186.2)
- added R313: 330k, Resistor_SMD:R_0402_1005Metric, F.Cu at (-191.4, 190.2)
- added R314: 2.2k, Resistor_SMD:R_0402_1005Metric, F.Cu at (-68.6, 9.68)
- added R315: 2.2k, Resistor_SMD:R_0402_1005Metric, F.Cu at (-68.6, 13.7)
- added R316: 10k 1%, Resistor_SMD:R_0402_1005Metric, F.Cu at (-68.6, 17.8)
- added R317: 220, Resistor_SMD:R_0402_1005Metric, F.Cu at (-68.6, 21.8)
- added R318: 75, Resistor_SMD:R_0402_1005Metric, F.Cu at (-68.6, 25.9)
- added R319: 10k 1%, Resistor_SMD:R_0402_1005Metric, F.Cu at (-68.6, 29.9)
- added R320: 220, Resistor_SMD:R_0402_1005Metric, F.Cu at (-68.6, 34.0)
- added R321: 75, Resistor_SMD:R_0402_1005Metric, F.Cu at (-68.6, 38.0)
- added R322: 3.3k, Resistor_SMD:R_0402_1005Metric, F.Cu at (-68.6, 42.1)
- added R323: 15k, Resistor_SMD:R_0402_1005Metric, F.Cu at (-68.6, 46.1)
- added R324: 3.3k, Resistor_SMD:R_0402_1005Metric, F.Cu at (-68.6, 50.2)
- added R325: 15k, Resistor_SMD:R_0402_1005Metric, F.Cu at (-68.6, 54.2)
- added R327: 33k, Resistor_SMD:R_0402_1005Metric, F.Cu at (78.8, 107.9)
- added R329: 6.8k, Resistor_SMD:R_0402_1005Metric, F.Cu at (78.8, 103.5)
- added R330: 3.3k, Resistor_SMD:R_0402_1005Metric, F.Cu at (78.8, 105.8)
- added R332: 3.3M, Resistor_SMD:R_0402_1005Metric, F.Cu at (-52.8, 5.63)
- added R334: 3.3M, Resistor_SMD:R_0402_1005Metric, F.Cu at (-52.8, 9.68)
- added R336: 1M, Resistor_SMD:R_0402_1005Metric, F.Cu at (79.1, 152.7)
- added R338: 4.7k, Resistor_SMD:R_0402_1005Metric, F.Cu at (-52.8, 17.8)
- added R339: 4.7k, Resistor_SMD:R_0402_1005Metric, F.Cu at (-52.8, 21.8)
- added R340: 10k, Resistor_SMD:R_0402_1005Metric, F.Cu at (-52.8, 25.9)
- added R341: 1k, Resistor_SMD:R_0402_1005Metric, F.Cu at (145.7, 74.1)
- added R342: 1k, Resistor_SMD:R_0402_1005Metric, F.Cu at (133.6, 74.1)
- added R343: 1k, Resistor_SMD:R_0402_1005Metric, F.Cu at (139.6, 74.1)
- added R344: 33k, Resistor_SMD:R_0402_1005Metric, F.Cu at (142.7, 74.1)
- added R345: 33k, Resistor_SMD:R_0402_1005Metric, F.Cu at (136.6, 74.1)
- added R346: 33k, Resistor_SMD:R_0402_1005Metric, F.Cu at (148.7, 74.1)
- added R347: 10, Resistor_SMD:R_0402_1005Metric, F.Cu at (140.8, 140.1)
- added R348: 10K, Resistor_SMD:R_0402_1005Metric, F.Cu at (135.6, 136.5)
- added W1: W, NetTie:NetTie-2_SMD_Pad0.5mm, F.Cu at (78.7, 98.6)
- added W2: W, NetTie:NetTie-2_SMD_Pad0.5mm, F.Cu at (78.7, 100.1)
- added W3: W, NetTie:NetTie-2_SMD_Pad0.5mm, F.Cu at (78.7, 101.6)
- added Y201: XO32, Oscillator:Oscillator_SMD_EuroQuartz_XO32-4Pin_3.2x2.5mm, F.Cu at (99.3, 76.5)
- C201, C202, C203, C204, C206, C207, C208, C209, C214, C215, C216, C217, C218, C219, C220, C221, C223, C224, C229, C230, C231, C232, C233, C234, C235, C236, C237, C239, C301, C302, C303, C307, C308, C309, C310, C311, C314, C315, C316, C317, C320, C321, C324, C325, C326, C327, C328: footprint Capacitor_THT:C_Disc_D5.0mm_W2.5mm_P5.00mm -> Capacitor_SMD:C_0402_1005Metric
- C211: footprint Capacitor_THT:CP_Radial_D8.0mm_P2.50mm -> Capacitor_SMD:CP_Elec_8x10.5
- C212, C213: footprint Capacitor_THT:CP_Radial_D8.0mm_P2.50mm -> Capacitor_SMD:CP_Elec_6.3x7.7
- C227: footprint Capacitor_THT:CP_Radial_Tantal_D5.5mm_P2.50mm -> Capacitor_SMD:C_1206_3216Metric
- C228: value 22uF 16V -> 22uF; footprint Capacitor_THT:CP_Radial_Tantal_D5.0mm_P2.50mm -> Capacitor_SMD:C_1206_3216Metric
- C304, C305, C306: value 10nF -> 4.7nF C0G; footprint Capacitor_THT:C_Disc_D7.5mm_W5.0mm_P5.00mm -> Capacitor_SMD:C_0603_1608Metric
- C312, C313: value 10nF -> 10nF C0G; footprint Capacitor_THT:C_Disc_D7.5mm_W5.0mm_P5.00mm -> Capacitor_SMD:C_0603_1608Metric
- C323: footprint Capacitor_THT:CP_Radial_D4.0mm_P2.00mm -> Capacitor_SMD:C_0805_2012Metric
- D201, D301, D302: footprint Diode_THT:D_DO-34_SOD68_P12.70mm_Horizontal -> Diode_SMD:D_SOD-123
- FB201, FB202: footprint Inductor_THT:L_Axial_L7.0mm_D3.3mm_P12.70mm_Horizontal_Fastron_MICC -> Inductor_SMD:L_0805_2012Metric
- IC201: value 2363 -> 27C512PLCC; footprint Package_DIP:DIP-28_W15.24mm -> Package_LCC:PLCC-32_THT-Socket
- IC204: value 2114 -> CY62256-70PC; footprint Package_DIP:DIP-18_W7.62mm -> Package_SO:SOP-28_8.4x18.16mm_P1.27mm
- IC206: value 68A09 -> MC6809E; footprint Package_DIP:DIP-40_W15.24mm -> Package_LCC:PLCC-44_SMD-Socket
- IC207: footprint Package_DIP:DIP-40_W15.24mm -> Package_LCC:PLCC-44_SMD-Socket
- IC208: value AY3-8912 -> YM2149; footprint Package_DIP:DIP-28_W15.24mm -> Package_DIP:DIP-40_W15.24mm_Socket
- IC301, IC302: footprint Package_DIP:DIP-16_W7.62mm -> Package_SO:SOIC-16_3.9x9.9mm_P1.27mm
- IC303, IC305: footprint Package_DIP:DIP-14_W7.62mm -> Package_SO:SOIC-14_3.9x8.7mm_P1.27mm
- IC304: footprint Package_DIP:DIP-8_W7.62mm -> Package_SO:SOIC-8_3.9x4.9mm_P1.27mm
- Q301, Q302, Q303: footprint Package_TO_SOT_THT:TO-92_Wide -> Package_TO_SOT_SMD:SOT-23
- R302, R333, R335: footprint Potentiometer_THT:Potentiometer_ACP_CA14-H5_Horizontal -> Potentiometer_THT:Potentiometer_Bourns_3296W_Vertical
- SW201: footprint TestPoint:TestPoint_Bridge_Pitch5.08mm_Drill1.3mm -> Connector_PinHeader_2.54mm:PinHeader_1x02_P2.54mm_Vertical
- moved C215 361.0 mm to (-251.8, 181.9)
- moved C216 361.0 mm to (-251.8, 186.0)
- moved C217 361.0 mm to (-251.8, 190.0)
- moved C218 361.0 mm to (-251.8, 194.1)
- moved C219 361.0 mm to (-251.8, 198.1)
- moved C220 361.0 mm to (-251.8, 202.2)
- moved C221 361.0 mm to (-251.8, 206.2)
- moved C230 361.0 mm to (-243.6, 190.0)
- moved C231 361.0 mm to (-243.6, 194.1)
- moved C232 361.0 mm to (-243.6, 198.1)
- moved C233 361.0 mm to (-243.6, 202.2)
- moved C234 361.0 mm to (-243.6, 206.2)
- moved C235 361.0 mm to (-243.6, 210.3)
- moved C236 361.0 mm to (-243.6, 214.3)
- moved C237 361.0 mm to (-243.6, 218.4)
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Connections:
- C323 pad 2: /CH(A+B+C)+DIGITAL_AUDIO -> /AUDIO
- IC201 pad 1: +5V -> unconnected-(IC201-NC-Pad1)
- IC201 pad 10: /A0 -> /A1
- IC201 pad 11: /D0 -> /A0
- IC201 pad 12: /D1 -> unconnected-(IC201-NC-Pad12)
- IC201 pad 13: /D2 -> /D0
- IC201 pad 14: GNDD -> /D1
- IC201 pad 15: /D3 -> /D2
- IC201 pad 16: /D4 -> GNDD
- IC201 pad 17: /D5 -> unconnected-(IC201-NC-Pad17)
- IC201 pad 18: /D6 -> /D3
- IC201 pad 19: /D7 -> /D4
- IC201 pad 2: /A12 -> /ROM_BANK2
- IC201 pad 20: /~{ROMS} -> /D5
- IC201 pad 21: /A10 -> /D6
- IC201 pad 22: /~{ROMOE} -> /D7
- IC201 pad 23: /A11 -> /~{ROMS}
- IC201 pad 24: /A9 -> /A10
- IC201 pad 25: /A8 -> /~{ROMOE}
- IC201 pad 27: +5V -> /A11
- IC201 pad 28: +5V -> /A9
- IC201 pad 3: /A7 -> /A12
- IC201 pad 4: /A6 -> /A7
- IC201 pad 5: /A5 -> /A6
- IC201 pad 6: /A4 -> /A5
- IC201 pad 7: /A3 -> /A4
- IC201 pad 8: /A2 -> /A3
- IC201 pad 9: /A1 -> /A2
- IC204 pad 1: /A6 -> GNDD
- IC204 pad 10: /RAM_R~{W} -> /A0
- IC204 pad 11: /D3 -> /D0
- IC204 pad 12: /D2 -> /D1
- IC204 pad 13: /D1 -> /D2
- IC204 pad 14: /D0 -> GNDD
- IC204 pad 15: /A9 -> /D3
- IC204 pad 16: /A8 -> /D4
- IC204 pad 17: /A7 -> /D5
- IC204 pad 18: +5V -> /D6
- IC204 pad 2: /A5 -> GNDD
- IC204 pad 3: /A4 -> /A7
- IC204 pad 4: /A3 -> /A6
- IC204 pad 5: /A0 -> /A5
- IC204 pad 6: /A1 -> /A4
- IC204 pad 7: /A2 -> /A3
- IC204 pad 8: /~{RAMS} -> /A2
- IC204 pad 9: GNDD -> /A1
- IC206 pad 33: Net-(IC206-~{DMA/BREQ}) -> unconnected-(IC206-BUSY-Pad33)
- IC206 pad 35: unconnected-(IC206-Q-Pad35) -> /Q
- IC206 pad 36: Net-(IC206-MRDY) -> unconnected-(IC206-AVMA-Pad36)
- IC206 pad 38: /EXTAL -> unconnected-(IC206-LIC-Pad38)
- IC206 pad 39: /XTAL -> GNDD
- IC208 pad 1: /CHC -> GNDD
- IC208 pad 10: /SW4 -> unconnected-(IC208-IOB3-Pad10)
- IC208 pad 11: /SW3 -> unconnected-(IC208-IOB2-Pad11)
- IC208 pad 12: /SW2 -> unconnected-(IC208-IOB1-Pad12)
- IC208 pad 13: /SW1 -> unconnected-(IC208-IOB0-Pad13)
- IC208 pad 14: /SW0 -> /SW7
- IC208 pad 15: /E -> /SW6
- IC208 pad 16: /~{RESET} -> /SW5
- IC208 pad 17: /BC2 -> /SW4
- IC208 pad 18: /BDIR -> /SW3
- IC208 pad 19: /BC2 -> /SW2
- IC208 pad 20: /BC1 -> /SW1
- IC208 pad 21: /P7 -> /SW0
- IC208 pad 22: /P6 -> /E
- IC208 pad 23: /P5 -> /~{RESET}
- IC208 pad 24: /P4 -> GNDD
- IC208 pad 25: /P3 -> +5V
- IC208 pad 26: /P2 -> +5V
- IC208 pad 27: /P1 -> /BDIR
- IC208 pad 28: /P0 -> /BC2
- IC208 pad 3: +5V -> /CHA
- IC208 pad 5: /CHA -> unconnected-(IC208-NC-Pad5)
- IC208 pad 6: GNDD -> unconnected-(IC208-IOB7-Pad6)
- IC208 pad 7: /SW7 -> unconnected-(IC208-IOB6-Pad7)
- IC208 pad 8: /SW6 -> unconnected-(IC208-IOB5-Pad8)
- IC208 pad 9: /SW5 -> unconnected-(IC208-IOB4-Pad9)
Other:
- board outline added: 80 x 130 mm

Commit message: Repro PCB: checkpoint - digital board placement + bus routing WIP
Two-board split layout: digital + analog regions. Big-chip cluster
(CPU/ROM/RAM) placed and oriented (data bus south), data+address bus
routed between them. J204 power connector, smaller-footprint pending.
Inter-board FFC+power-header strategy defined. 4-layer ground/power
zones next. Schematic complete; PCB layout in progress.

Co-Authored-By: Claude Opus 4.8 <noreply@anthropic.com>
Parts:
- J204: footprint Connector_Molex:Molex_KK-396_A-41791-0004_1x04_P3.96mm_Vertical -> Connector_JST:JST_PH_B4B-PH-K_1x04_P2.00mm_Vertical
- moved R311 437.9 mm to (225.4, 105.2)
- moved C307 421.1 mm to (229.0, 119.8)
- moved C315 414.9 mm to (229.3, 118.2)
- moved C317 409.5 mm to (225.3, 119.4)
- moved C316 407.0 mm to (225.4, 100.9)
- moved C327 405.9 mm to (229.4, 101.1)
- moved J301 405.0 mm to (180.0, 140.9)
- moved C326 402.5 mm to (225.3, 99.4)
- moved MNT4 384.2 mm to (220.1, 33.2)
- moved D302 382.8 mm to (216.2, 126.7), turned to -90 degrees
- moved C328 381.7 mm to (198.0, 129.7), turned to 90 degrees
- moved C302 381.0 mm to (190.8, 99.4)
- moved C303 380.7 mm to (191.0, 101.7)
- moved C301 379.3 mm to (190.6, 96.6)
- moved MNT3 376.5 mm to (213.4, 33.2)
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Connections:
- net /CH(A+B+C) renamed Net-(C323-Pad1)
Routing:
- net /D2: track 0.00 -> 219.5 mm, vias 0 -> 4
- net /D0: track 0.00 -> 197.0 mm, vias 0 -> 4
- net /A12: track 0.00 -> 188.9 mm, vias 0 -> 6
- net /D1: track 0.00 -> 187.4 mm, vias 0 -> 5
- net /D4: track 0.00 -> 180.4 mm, vias 0 -> 4
- net /D3: track 0.00 -> 179.4 mm, vias 0 -> 4
- net /D6: track 0.00 -> 174.2 mm, vias 0 -> 4
- net /D5: track 0.00 -> 167.8 mm, vias 0 -> 4
- net /E: track 0.00 -> 150.7 mm, vias 0 -> 3
- net /A8: track 0.00 -> 147.7 mm, vias 0 -> 5
- net /D7: track 0.00 -> 147.4 mm, vias 0 -> 3
- net /A9: track 0.00 -> 146.7 mm, vias 0 -> 4
- net /R~{W}: track 0.00 -> 133.8 mm, vias 0 -> 2
- net /~{NMI}: track 0.00 -> 130.9 mm, vias 0 -> 3
- net /A7: track 0.00 -> 122.7 mm, vias 0 -> 5
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Other:
- board size 80 x 130 mm -> 208.4 x 105 mm
- copper layers 2 -> 4
